File: RS485-Transceiver.kicad_sch (KiCad schematic)
At the start: 7 parts, among them J2 G800W306018EU, U19 ISOW1412DFM

Commit message: v1.0 ordered
Parts:
- C1, C2: footprint C0402C103K3REC7411:CAPC10555_55N_KEM -> CAPC10555_55N_KEM; LCSC (none) -> C650944
- C3, C4: footprint GRM155R61A:CAP_GRM155R61A106ME11_MUR -> CAP_GRM155R61A106ME11_MUR; LCSC (none) -> C408132
- J2: footprint G800W306018EU:CONN02_G800_5P08X2P5_AMP -> CONN02_G800_5P08X2P5_AMP; LCSC (none) -> C5360898
- R1: footprint ERJ_PA2F1200X:RES_ERJPA2F1200X -> ERJPA2F1200X:RES_ERJPA2F1200X; LCSC (none) -> C102779
- U19: footprint footprints:DFM0020A-IPC_A -> DFM0020A-IPC_A; LCSC (none) -> C5216548
Changed lines of the file:
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@@
 			)
 		)
-		(property "Description" ""
+		(property "Description" "Power symbol creates a global label with name \"+3.3V\""
 			(at 80.01 63.5 0)
 			(effects
@@
 			)
 		)
-		(property "Footprint" "C0402C103K3REC7411:CAPC10555_55N_KEM"
+		(property "Footprint" "CAPC10555_55N_KEM"
 			(at 172.72 78.74 0)
 			(effects
@@
 		)
 		(property "Description" "C0402C103K3REC7411"
+			(at 172.72 78.74 0)
+			(effects
+				(font
+					(size 1.27 1.27)
+				)
+				(hide yes)
+			)
+		)
+		(property "LCSC" "C650944"
 			(at 172.72 78.74 0)
 			(effects
@@
 			)
 		)
-		(property "Footprint" "G800W306018EU:CONN02_G800_5P08X2P5_AMP"
+		(property "Footprint" "CONN02_G800_5P08X2P5_AMP"
 			(at 227.33 93.98 0)
 			(effects
@@
 			)
 		)
+		(property "LCSC" "C5360898"
+			(at 227.33 93.98 0)
+			(effects
+				(font
+					(size 1.27 1.27)
+				)
+				(hide yes)
+			)
+		)
 		(pin "1"
 		)
@@
 			)
 		)
-		(property "Description" ""
+		(property "Description" "Power symbol creates a global label with name \"+5V\""
 			(at 104.14 63.5 0)
 			(effects
@@
 			)
 		)
-		(property "Footprint" "C0402C103K3REC7411:CAPC10555_55N_KEM"
+		(property "Footprint" "CAPC10555_55N_KEM"
 			(at 104.14 78.74 0)
 			(effects
@@
 		)
 		(property "Description" "C0402C103K3REC7411"
+			(at 104.14 78.74 0)
+			(effects
+				(font
+					(size 1.27 1.27)
+				)
+				(hide yes)
+			)
+		)
+		(property "LCSC" "C650944"
 			(at 104.14 78.74 0)
 			(effects
@@
 			)
 		)
-		(property "Footprint" "footprints:DFM0020A-IPC_A"
+		(property "Footprint" "DFM0020A-IPC_A"
 			(at 121.92 73.66 0)
 			(effects
@@
 				)
 				(hide yes)
+			)
+		)
+		(property "LCSC" "C5216548"
+			(at 121.92 73.66 0)
+			(effects
+				(font
+					(size 1.27 1.27)
+				)
 			)
 		)
@@
 			)
 		)
-		(property "Footprint" "GRM155R61A:CAP_GRM155R61A106ME11_MUR"
+		(property "Footprint" "CAP_GRM155R61A106ME11_MUR"
 			(at 91.44 78.74 0)
 			(effects
@@
 			)
 		)
-		(property "Description" "GRM155R61A106ME11D"
+		(property "Description" "10uF, 10V"
+			(at 91.44 78.74 0)
+			(effects
+				(font
+					(size 1.27 1.27)
+				)
+				(hide yes)
+			)
+		)
+		(property "LCSC" "C408132"
 			(at 91.44 78.74 0)
 			(effects
@@
 			)
 		)
-		(property "Footprint" "ERJ_PA2F1200X:RES_ERJPA2F1200X"
+		(property "Footprint" "ERJPA2F1200X:RES_ERJPA2F1200X"
 			(at 227.33 114.3 0)
 			(effects
@@
 				)
 				(justify bottom)
+				(hide yes)
+			)
+		)
+		(property "LCSC" "C102779"
+			(at 227.33 114.3 0)
+			(effects
+				(font
+					(size 1.27 1.27)
+				)
 				(hide yes)
 			)
@@
 			)
 		)
-		(property "Footprint" "GRM155R61A:CAP_GRM155R61A106ME11_MUR"
+		(property "Footprint" "CAP_GRM155R61A106ME11_MUR"
 			(at 186.69 78.74 0)
 			(effects
@@
 			)
 		)
-		(property "Description" "GRM155R61A106ME11D"
+		(property "Description" "10uF, 10V"
 			(at 186.69 78.74 0)
 			(effects
+				(font
+					(size 1.27 1.27)
+				)
+				(hide yes)
+			)
+		)
+		(property "LCSC" "C408132"
+			(at 186.69 78.74 0)
+			(effects
