File: TPM-IO-BOARD.kicad_pcb (KiCad board)
At the start: 4 copper layers, 95 x 58 mm, 107 parts, among them J1 GPIO, J10 691322110002, J11 691322110002, J12 691322110002, J13 691322110002, J14 691322110002, J15 691322110002, J16 1844223, J17 1844223, J18 1844223, J2 G800W306018EU, J3 691322110002, J4 691322110002, J5 691322110002, J6 691322110002, J7 691322110002, J8 691322110002, J9 691322110002, Q1 2N7002NXAKR, Q10 2N7002NXAKR, Q11 2N7002NXAKR, Q12 2N7002NXAKR, Q2 2N7002NXAKR, Q3 2N7002NXAKR, Q4 2N7002NXAKR, Q5 2N7002NXAKR, Q6 2N7002NXAKR, Q7 2N7002NXAKR, Q8 2N7002NXAKR, Q9 2N7002NXAKR, U19 ISOW1412DFM, U32 AQY212EHAX, U7 AQY212EHAX

Commit message: v1.0 ordered
Parts:
- added C5: 470uF, 35ZLH470MEFC10X16:CAP_YX_10X16_RUB, F.Cu at (168.2, 48.5)
- added C6: 470uF, 35ZLH470MEFC10X16:CAP_YX_10X16_RUB, F.Cu at (168.2, 60.0)
- added C7: 470uF, 35ZLH470MEFC10X16:CAP_YX_10X16_RUB, F.Cu at (168.2, 71.8)
- added LED12: SZYY0402YG, 150040V:LED_S73240_WRE, F.Cu at (136.8, 59.8)
- added LED14: SZYY0402YG, 150040V:LED_S73240_WRE, F.Cu at (136.8, 62.2)
- added LED15: SZYY0402YG, 150040V:LED_S73240_WRE, F.Cu at (136.8, 64.5)
- added R42: 1k, RC0402JR_071KL:RC0402N_YAG, F.Cu at (139.2, 62.2)
- added R43: SMD-RES-10K-5_-1__0402_, RC0402JR_0710KL:R0402, F.Cu at (139.2, 64.5)
- added R44: 330, RC0402FR_07330RL:RESC1005X40N, F.Cu at (139.2, 59.8)
Routing:
- net /GPIO20/PCM.DIN: track 37.0 -> 78.7 mm, vias 0 -> 1
- net +24V: track 89.9 -> 123.3 mm, vias 16 -> 18
- net BUS_GND: track 37.7 -> 71.0 mm, vias 13 -> 15
- net /GPIO26: track 32.4 -> 64.2 mm
- net +5V: track 32.1 -> 62.2 mm
- net /GPIO16: track 41.9 -> 62.3 mm
- net /GPIO19/PCM.FS: track 45.0 -> 59.7 mm
- net /GPIO13/PWM1: track 53.8 -> 68.1 mm
- net /GPIO12/PWM0: track 52.8 -> 64.2 mm
- net /GPIO6: track 46.6 -> 55.2 mm
- net +3V3: track 14.2 -> 19.7 mm, vias 4 -> 5
- net /GPIO5: track 44.2 -> 49.5 mm
- net GND: track 25.7 -> 27.6 mm, vias 18 -> 20
- net Net-(LED15-Pad2): track 0.00 -> 1.51 mm
- net Net-(LED12-Pad2): track 0.00 -> 1.45 mm
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Other:
- board text added: "24V"
- board text added: "3V3"
- board text added: "5V"
- board text added: "IN1"
- board text added: "IN2"
- board text added: "MODBUS"
- board text added: "SOL1"
- board text added: "SOL10"
- board text added: "SOL11"
- board text added: "SOL12"
- board text added: "SOL2"
- board text added: "SOL3"
- board text added: "SOL4"
- board text added: "SOL5"
- board text added: "SOL6"
- board text added: "SOL7"
- board text added: "SOL8"
- board text added: "SOL9"
