File: TPM-IO-BOARD.kicad_sch (KiCad schematic)
At the start: 18 parts, among them J1 GPIO, J10 691322110002, J11 691322110002, J12 691322110002, J13 691322110002, J14 691322110002, J15 691322110002, J16 1844223, J17 1844223, J18 1844223, J3 691322110002, J4 691322110002, J5 691322110002, J6 691322110002, J7 691322110002, J8 691322110002, J9 691322110002

Commit message: v1.0 ordered
Parts:
- added C5, C6, C7: 470uF, CAP_YX_10X16_RUB, symbol 35ZLH470MEFC10X16:35ZLH470MEFC10X16
- J1: LCSC (none) -> C35165
- J10, J11, J12, J13, J14, J15, J3, J4, J5, J6, J7, J8, J9: LCSC (none) -> C61791
- J16, J17, J18: footprint 1844223:CONN_1844223_PXC -> CONN_1844223_PXC; LCSC (none) -> C5244104
Connections:
- net +24V: now also C5.1, C6.1, C7.1
- net BUS_GND: now also C5.2, C6.2, C7.2
Other:
- added sheet LED-Indicators (untitled.kicad_sch)
- note added: "Bus Capacitance"
- note added: "Vbus In"
