File: opto-isolator.kicad_sch (KiCad schematic)
At the start: 3 parts, among them U32 AQY212EHAX

Commit message: v1.0 ordered
Parts:
- R40, R41: footprint RC0402JR_0710KL:R0402 -> SMD-RES-10K-5_-1__0402_:R0402; LCSC (none) -> C319934
- U32: footprint OptoDevice:Panasonic_APV-AQY_SSOP-4_4.45x2.65mm_P1.27mm -> RELAY_AQY_SO4_EH_PAN; LCSC (none) -> C29276
Changed lines of the file:
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@@
 			)
 		)
-		(property "Description" ""
+		(property "Description" "Power symbol creates a global label with name \"+3.3V\""
 			(at 171.45 71.12 0)
 			(effects
@@
 			)
 		)
-		(property "Footprint" "RC0402JR_0710KL:R0402"
+		(property "Footprint" "SMD-RES-10K-5_-1__0402_:R0402"
 			(at 95.25 87.63 0)
 			(effects
@@
 				)
 				(justify bottom)
+			)
+		)
+		(property "LCSC" "C319934"
+			(at 95.25 87.63 0)
+			(effects
+				(font
+					(size 1.27 1.27)
+				)
+				(hide yes)
 			)
 		)
@@
 			)
 		)
-		(property "Footprint" "OptoDevice:Panasonic_APV-AQY_SSOP-4_4.45x2.65mm_P1.27mm"
+		(property "Footprint" "RELAY_AQY_SO4_EH_PAN"
 			(at 118.11 87.63 0)
 			(effects
@@
 				)
 				(hide yes)
+			)
+		)
+		(property "LCSC" "C29276"
+			(at 118.11 87.63 0)
+			(effects
+				(font
+					(size 1.27 1.27)
+				)
 			)
 		)
@@
 			)
 		)
-		(property "Footprint" "RC0402JR_0710KL:R0402"
+		(property "Footprint" "SMD-RES-10K-5_-1__0402_:R0402"
 			(at 171.45 80.01 0)
 			(effects
@@
 			)
 		)
+		(property "LCSC" "C319934"
+			(at 171.45 80.01 0)
+			(effects
+				(font
+					(size 1.27 1.27)
+				)
+				(hide yes)
+			)
+		)
