File: solenoid-driver.kicad_sch (KiCad schematic)
At the start: 6 parts, among them Q10 2N7002NXAKR

Commit message: v1.0 ordered
Parts:
- D10: LCSC (none) -> C328592
- LED9: LCSC (none) -> C264407
- Q10: footprint KiCad:SOT95P230X110-3N -> SOT95P230X110-3N; LCSC (none) -> C414015; Manufacturer_Part_Number 2N7002NXAKR -> 2N7002K
- R28: footprint RC0402FR_07330RL:RESC1005X40N -> RC0402FR-07330RL:RESC1005X40N; LCSC (none) -> C517531
- R29, R30: footprint RC0402JR_0710KL:R0402 -> SMD-RES-10K-5_-1__0402_:R0402; LCSC (none) -> C319934
Changed lines of the file:
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@@
 			)
 		)
-		(property "Footprint" "RC0402FR_07330RL:RESC1005X40N"
+		(property "Footprint" "RC0402FR-07330RL:RESC1005X40N"
 			(at 95.25 99.06 0)
 			(effects
@@
 		)
 		(property "Description" "RC0402FR-07330RL"
+			(at 95.25 99.06 0)
+			(effects
+				(font
+					(size 1.27 1.27)
+				)
+				(hide yes)
+			)
+		)
+		(property "LCSC" "C517531"
 			(at 95.25 99.06 0)
 			(effects
@@
 			)
 		)
+		(property "LCSC" "C264407"
+			(at 154.94 68.58 0)
+			(effects
+				(font
+					(size 1.27 1.27)
+				)
+				(hide yes)
+			)
+		)
 		(pin "1"
 		)
@@
 			)
 		)
+		(property "LCSC" "C328592"
+			(at 190.5 59.69 0)
+			(effects
+				(font
+					(size 1.27 1.27)
+				)
+				(hide yes)
+			)
+		)
 		(pin "2"
 		)
@@
 			)
 		)
-		(property "Footprint" "KiCad:SOT95P230X110-3N"
+		(property "Footprint" "SOT95P230X110-3N"
 			(at 149.86 197.79 0)
 			(effects
@@
 			)
 		)
-		(property "Manufacturer_Part_Number" "2N7002NXAKR"
+		(property "Manufacturer_Part_Number" "2N7002K"
 			(at 149.86 897.79 0)
 			(effects
@@
 				)
 				(justify left top)
+				(hide yes)
+			)
+		)
+		(property "LCSC" "C414015"
+			(at 138.43 99.06 0)
+			(effects
+				(font
+					(size 1.27 1.27)
+				)
 				(hide yes)
 			)
@@
 			)
 		)
-		(property "Footprint" "RC0402JR_0710KL:R0402"
+		(property "Footprint" "SMD-RES-10K-5_-1__0402_:R0402"
 			(at 154.94 64.77 0)
 			(effects
@@
 				)
 				(justify bottom)
+			)
+		)
+		(property "LCSC" "C319934"
+			(at 154.94 64.77 0)
+			(effects
+				(font
+					(size 1.27 1.27)
+				)
+				(hide yes)
 			)
 		)
@@
 			)
 		)
-		(property "Footprint" "RC0402JR_0710KL:R0402"
+		(property "Footprint" "SMD-RES-10K-5_-1__0402_:R0402"
 			(at 121.92 109.22 0)
 			(effects
@@
 			)
 		)
+		(property "LCSC" "C319934"
+			(at 121.92 109.22 0)
+			(effects
+				(font
+					(size 1.27 1.27)
+				)
+				(hide yes)
+			)
+		)
